File: KiCad/TeamProject/Leader.kicad_sch (KiCad schematic)
At the start: 9 parts, among them SW1 Reset, U1 PIC32MX170F256B

Commit message: Merge branch 'main' of https://github.com/ttyaaron/ME218B_TeamProject
# Conflicts:
#	LeaderPIC.X/ProjectSource/CommonDefinitions.c
#	LeaderPIC.X/build/default/debug/ProjectSource/BeaconDetectFSM.o
#	LeaderPIC.X/build/default/debug/ProjectSource/CommonDefinitions.o
#	LeaderPIC.X/build/default/debug/ProjectSource/DCMotorService.o
#	LeaderPIC.X/build/default/debug/ProjectSource/EventCheckers.o
#	LeaderPIC.X/build/default/debug/ProjectSource/MainLogicFSM.o
#	LeaderPIC.X/build/default/debug/ProjectSource/SPILeaderFSM.o
#	LeaderPIC.X/build/default/debug/ProjectSource/TestHarnessService0.o
#	LeaderPIC.X/build/default/production/ProjectSource/BeaconDetectFSM.o
#	LeaderPIC.X/build/default/production/ProjectSource/CommonDefinitions.o
#	LeaderPIC.X/build/default/production/ProjectSource/DCMotorService.o
#	LeaderPIC.X/build/default/production/ProjectSource/EventCheckers.o
#	LeaderPIC.X/build/default/production/ProjectSource/MainLogicFSM.o
#	LeaderPIC.X/build/default/production/ProjectSource/SPILeaderFSM.o
#	LeaderPIC.X/build/default/production/ProjectSource/TestHarnessService0.o
#	LeaderPIC.X/dist/default/debug/LeaderPIC.X.debug.elf
#	LeaderPIC.X/dist/default/debug/LeaderPIC.X.debug.map
#	LeaderPIC.X/dist/default/debug/memoryfile.xml
#	LeaderPIC.X/dist/default/production/LeaderPIC.X.production.elf
#	LeaderPIC.X/dist/default/production/LeaderPIC.X.production.hex
#	LeaderPIC.X/dist/default/production/LeaderPIC.X.production.map
#	LeaderPIC.X/dist/default/production/memoryfile.xml
Parts:
- added U2, U5: Quadrature_Encoder, symbol ME218_BaseLib:Quadrature_Encoder
Connections:
- net +3.3V: now also U2.1 (Vcc), U5.1 (Vcc)
- net Left Encoder IC1: now also U2.2 (ChA)
- net Right Encoder IC2: now also U5.2 (ChA)
- new net GND: U2.4 (GND), U5.4 (GND)
